Commit message: new world + new camera

File: src/kobuki/kobuki_description/urdf/kobuki.urdf.xacro (robot description, xacro)
@@ -222,5 +222,5 @@
     <joint name="camara_profundidad_joint" type="fixed">
       <!--axis xyz="0 1 0" /-->
-      <origin xyz="0.12 0 1.5" rpy="0 0 0" />  <!--heght480-640/2-->
+      <origin xyz="0.05 0 1.5" rpy="0 0 0" />  <!--heght480-640/2-->
       <!--parent link="base_link"/-->
       <!--parent link="pc_base_up"/-->
@@ -264,4 +264,20 @@
       </visual>
     </link>
+    <link name="camara_rgb">
+      <visual>
+        <origin xyz="0 0 0" rpy="0 0 0"/>
+        <geometry>
+          <!--mesh filename="package://kobuki_description/meshes/camera_ASUS_XTION.STL"/-->
+          <box size="0.08 0.08 0.08"/>
+          <!--box size="0 0 0"/-->
+        </geometry>
+        <material name="red"/>
+      </visual>
+    </link>
+    <joint name="camara_rgb_joint" type="fixed">
+      <origin xyz="0 0 1.5" rpy="0 0 0" />
+      <parent link="base_link" />
+      <child link="camara_rgb" />
+    </joint>
     <!--agrega laser hokuyo-->
     <link name="hokuyo_link" type="fixed">

File: src/kobuki/kobuki_description/urdf/kobuki_gazebo.urdf.xacro (robot description, xacro)
@@ -103,5 +103,5 @@
             <clip>
                 <near>0.3</near>
-                <far>2</far>
+                <far>20</far>
             </clip>
         </camera>
@@ -220,4 +220,47 @@
 	    </sensor>
 	  </gazebo>
+		<!-- camera -->
+	  <gazebo reference="camara_rgb">
+		<sensor type="camera" name="camera1">
+			<update_rate>30.0</update_rate>
+			<camera name="head">
+			<save enabled="true">
+				<path>/home/rafael/PAI/images</path>
+			</save>
+			<horizontal_fov>1.3962634</horizontal_fov>
+			<image>
+				<width>800</width>
+				<height>800</height>
+				<format>R8G8B8</format>
+			</image>
+			<clip>
+				<near>0.02</near>
+				<far>300</far>
+			</clip>
+			<noise>
+				<type>gaussian</type>
+				<!-- Noise is sampled independently per pixel on each frame.
+					That pixel's noise value is added to each of its color
+					channels, which at that point lie in the range [0,1]. -->
+				<mean>0.0</mean>
+				<stddev>0.007</stddev>
+			</noise>
+			</camera>
+			<plugin name="camera_controller" filename="libgazebo_ros_camera.so">
+			<alwaysOn>true</alwaysOn>
+			<updateRate>0.0</updateRate>
+			<cameraName>rrbot/camera1</cameraName>
+			<imageTopicName>image_raw</imageTopicName>
+			<cameraInfoTopicName>camera_info</cameraInfoTopicName>
+			<frameName>camera_link</frameName>
+			<hackBaseline>0.07</hackBaseline>
+			<distortionK1>0.0</distortionK1>
+			<distortionK2>0.0</distortionK2>
+			<distortionK3>0.0</distortionK3>
+			<distortionT1>0.0</distortionT1>
+			<distortionT2>0.0</distortionT2>
+			</plugin>
+		</sensor>
+	  </gazebo>
 	  <gazebo reference="gyro_link">
 	   <sensor type="imu" name="imu">
